File: v2.1-desktop/otter-iron-pro-v2.1-desktop/v2-bottom.sch (KiCad schematic (older format))
At the start: 0 parts

Commit message: Import v2.0 schematics
Parts:
- added C1, C11, C4, C9: 1μF 25V, otter:C_0603, symbol Device:C
- added C10, C18, C2, C5, C7, C8: 0.1μF, otter:C_0402, symbol Device:C
- added C16: 18p, otter:C_0402, symbol Device:C_Small
- added C17: DNP, otter:C_0402, symbol Device:C_Small
- added C22: 0.1μF, otter:C_0402, symbol Device:C_Small
- added C24: 1000µF, otter:CP_Radial_D10.0mm_P5.00mm_flat, symbol Device:CP_Small
- added D3: B140-E3, Diode_SMD:D_SOD-123F, symbol Diode:B140-E3
- added J1: Conn_01x10, Connector_PinHeader_2.00mm:PinHeader_1x10_P2.00mm_Horizontal, symbol Connector_Generic:Conn_01x10
- added J3: C245, Connector_PinHeader_2.54mm:PinHeader_1x04_P2.54mm_Horizontal, symbol Connector:Conn_01x04_Male
- added L1: 4.7u, Inductor_SMD:L_Taiyo-Yuden_NR-60xx, symbol Device:L
- added NT1: JUNC_N, NetTie:NetTie-2_SMD_Pad0.5mm, symbol Device:Net-Tie_2
- added P1: TC2030-CTX, otter:TC2030, symbol OtterIron_Devkit-rescue:TC2030-CTX-Tag-Connect-pd-buddy-sink-rescue-usb-c-otter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
- added Q1, Q3: SS8050, Package_TO_SOT_SMD:SOT-23, symbol Transistor_BJT:MMBT3904
- added Q2: DMP3017SFG, otter:Diodes_PowerDI3333-8, symbol OtterIron_Devkit-rescue:DMP3017SFG-pd-buddy-pd-buddy-sink-rescue-pd-buddy-sink-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
- added Q4: BC807, Package_TO_SOT_SMD:SOT-23, symbol Transistor_BJT:BC807
- added R1: 560k, otter:R_0402, symbol Device:R_Small
- added R12, R14, R16, R18, R25, R5, R6, R9: 2k37, otter:R_0402, symbol Device:R
- added R15: 750k, otter:R_0402, symbol Device:R
- added R17: 100k, otter:R_0402, symbol Device:R
- added R19: 20, otter:R_0603, symbol Device:R
- added R2: 100k, otter:R_0402, symbol Device:R_Small
- added R20, R21: 33, otter:R_0402, symbol Device:R
- added R22: 10m, otter:R_0805, symbol Device:R_Small
- added R8: 2k37, otter:R_0402, symbol Device:R_Small
- added U2: AP2204R-3.3, Package_TO_SOT_SMD:SOT-89-3, symbol Regulator_Linear:AP2204R-3.3
- added U4: STM32F072C8Tx, otter:LQFP-48_7x7mm_P0.5mm, symbol MCU_ST_STM32F0:STM32F072C8Tx
- added U5: OPA340NA, Package_TO_SOT_SMD:SOT-23-5, symbol Amplifier_Operational:OPA340NA
- added U6: MCP9700AT-ETT, Package_TO_SOT_SMD:SOT-23, symbol Sensor_Temperature:MCP9700AT-ETT
- added U7: SI8540, Package_TO_SOT_SMD:SOT-23-5, symbol otter:SI8540
Connections:
- net labels added: +3V3, C245_JUNC, GND, IIN, INT_N, OLED_SCL, OLED_SDA, PWM, SW1, SW2, SWCLK, SWDIO, TREF, TTIP, UIN, USB_N, USB_P, VBUS, nRST
- wire segments 0 -> 150
