File: v2.1-desktop/otter-iron-pro-v2.1-desktop/v2-top.sch (KiCad schematic (older format))
At the start: 0 parts

Commit message: Import v2.0 schematics
Parts:
- added C12, C13, C14, C15, C19, C20: 1μF 25V, otter:C_0603, symbol Device:C
- added C21: 0.1μF, otter:C_0603, symbol Device:C
- added J1: USB_C_Receptacle_USB2.0, otter:USB-C 16Pin, symbol Connector:USB_C_Receptacle_USB2.0
- added J10, J3, J4, J7, J8, J9: Conn_01x01, otter:pad_1_2, symbol Connector_Generic:Conn_01x01
- added J11, J12, J13, J14, J15, J16: Conn_01x01, otter:pad_1.5_3, symbol Connector_Generic:Conn_01x01
- added J2: OLED_64x32, otter:0.69OLED, symbol Connector_Generic:Conn_01x14
- added J5, J6: Conn_01x01, otter:pad_0.75_3, symbol Connector_Generic:Conn_01x01
- added R10, R13, R23, R24, R7: 2k37, otter:R_0603, symbol Device:R
- added R11: 560k, otter:R_0603, symbol Device:R_Small
- added SW1: key1, Button_Switch_SMD:SW_SPST_EVQP7C, symbol Switch:SW_Push
- added SW2: key2, Button_Switch_SMD:SW_SPST_EVQP7C, symbol Switch:SW_Push
- added U1: USBLC6-4SC6, Package_TO_SOT_SMD:SOT-23-6, symbol OtterIron_PRO_Top-rescue:USBLC6-2SC6-Power_Protection
- added U3: STUSB4500QTR, otter:QFN-24-1EP_4x4mm_P0.5mm_EP2.7x2.7mm, symbol OtterIron_PRO_Top-rescue:STUSB4500-otter
Connections:
- net labels added: +3V3, CC1, CC2, GND, INT_N, OLED_SCL, OLED_SDA, SW1, SW2, USB_N, USB_P, VBUS
- wire segments 0 -> 56
- no-connect marks 0 -> 14
