File: v2.1-desktop/otter-iron-pro-v2.1-desktop/otter-iron-pro-v2.1-desktop.sch (KiCad schematic (older format))
At the start: 0 parts

Commit message: Consolidate schematics into a single sheet
Parts:
- added C? (x10): 1μF 25V, otter:C_0603, symbol Device:C
- added C?: 0.1μF, otter:C_0603, symbol Device:C
- added C? (x6): 0.1μF, otter:C_0402, symbol Device:C
- added C?: DNP, otter:C_0402, symbol Device:C_Small
- added C?: 18p, otter:C_0402, symbol Device:C_Small
- added C?: 0.1μF, otter:C_0402, symbol Device:C_Small
- added C?: 1000µF, otter:CP_Radial_D10.0mm_P5.00mm_flat, symbol Device:CP_Small
- added C?: DNP, symbol Device:C
- added C?: DNP, symbol Device:CP
- added D?: B140-E3, Diode_SMD:D_SOD-123F, symbol Diode:B140-E3
- added F?: Fuse, symbol Device:Fuse
- added J?: C245, otter:RPC1-12RB-6P(71), symbol Connector:Conn_01x06_Male
- added J?: OLED_64x32, otter:0.69OLED, symbol Connector_Generic:Conn_01x14
- added J?: USB_C_Receptacle_USB2.0, otter:USB-C 16Pin, symbol Connector:USB_C_Receptacle_USB2.0
- added J?: SWD, symbol Connector:Conn_01x03_Female
- added J? (x2): +24V, symbol Connector:Screw_Terminal_01x01
- added J?: SSD1306, Connector_PinHeader_2.54mm:PinHeader_1x04_P2.54mm_Vertical, symbol Connector:Conn_01x04_Male
- added L?: 4.7u, Inductor_SMD:L_Taiyo-Yuden_NR-60xx, symbol Device:L
- added NT?: JUNC_N, NetTie:NetTie-2_SMD_Pad0.5mm, symbol Device:Net-Tie_2
- added Q?: DMP3017SFG, otter:Diodes_PowerDI3333-8, symbol OtterIron_Devkit-rescue:DMP3017SFG-pd-buddy-pd-buddy-sink-rescue-pd-buddy-sink-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
- added Q? (x2): SS8050, Package_TO_SOT_SMD:SOT-23, symbol Transistor_BJT:MMBT3904
- added Q?: BC807, Package_TO_SOT_SMD:SOT-23, symbol Transistor_BJT:BC807
- added R?: 560k, otter:R_0603, symbol Device:R_Small
- added R? (x5): 2k37, otter:R_0603, symbol Device:R
- added R? (x8): 2k37, otter:R_0402, symbol Device:R
- added R?: 100k, otter:R_0402, symbol Device:R_Small
- added R?: 560k, otter:R_0402, symbol Device:R_Small
- added R?: 100k, otter:R_0402, symbol Device:R
- added R?: 750k, otter:R_0402, symbol Device:R
- added R?: 33, otter:R_0603, symbol Device:R
- added R? (x2): 33, otter:R_0402, symbol Device:R
- added R?: 10m, otter:R_0805, symbol Device:R
- added R?: 2k37, otter:R_0402, symbol Device:R_Small
- added SW?: key1, Button_Switch_SMD:SW_SPST_EVQP7C, symbol Switch:SW_Push
- added SW?: key2, Button_Switch_SMD:SW_SPST_EVQP7C, symbol Switch:SW_Push
- added U?: USBLC6-4SC6, Package_TO_SOT_SMD:SOT-23-6, symbol Power_Protection:USBLC6-4SC6
- added U?: STUSB4500QTR, otter:QFN-24-1EP_4x4mm_P0.5mm_EP2.7x2.7mm, symbol Interface_USB:STUSB4500QTR
- added U?: AP2204R-3.3, Package_TO_SOT_SMD:SOT-89-3, symbol Regulator_Linear:AP2204R-3.3
- added U?: OPA340NA, Package_TO_SOT_SMD:SOT-23-5, symbol Amplifier_Operational:OPA340NA
- added U?: MCP9700AT-ETT, Package_TO_SOT_SMD:SOT-23, symbol Sensor_Temperature:MCP9700AT-ETT
- added U?: STM32F072C8Tx, otter:LQFP-48_7x7mm_P0.5mm, symbol MCU_ST_STM32F0:STM32F072C8Tx
- added U?: SI8540, Package_TO_SOT_SMD:SOT-23-5, symbol SI8540:SI8540
Connections:
- new net: C?.1, C?.1, J?.5 (Pin_5), L?.2
- new net: C?.2, J?.1 (Pin_1)
- new net: J?.12 (Pin_12), R?.1
- new net: C?.1, J?.13 (Pin_13)
- new net: C?.1, J?.14 (Pin_14)
- new net: C?.1, J?.2 (Pin_2)
- new net: C?.1, J?.3 (Pin_3)
- new net: C?.2, J?.4 (Pin_4)
- new net: J?.9 (Pin_9), R?.1
- new net: C?.1, U?.23 (VREG_2V7)
- new net: C?.2, U?.21 (VREG_1V2)
- new net: R?.2, U?.18 (VBUS_VS_DISCH)
- new net: R?.2, U?.6 (RESET)
- new net: C?.1, Q?.1 (S), Q?.2 (S), Q?.3 (C), Q?.3 (S), R?.1, R?.2, R?.2
- new net: Q?.4 (G), R?.2
- new net: D?.1 (K), L?.1, Q?.5 (D)
- new net: Q?.3 (C), R?.1, R?.2
- new net: Q?.1 (B), R?.2
- new net: C?.2, R?.1, R?.2, U?.1
- new net: R?.2, U?.3 (+)
- new net: C?.1, R?.1, R?.2, U?.4 (-)
- new net: C?.1, NT?.1, R?.1
- new net: R?.2, U?.2 (Vout)
- new net: Q?.2 (E), Q?.2 (E), R?.1
- new net: R?.2, U?.1 (RG1)
- new net: R?.1, U?.5 (RG2)
- new net: Q?.1 (B), Q?.1 (B), R?.2
- new net: F?.2, J?.1 (Pin_1)
- new net +3V3: C?.1, C?.1, C?.1, C?.1, C?.1, C?.1, C?.1, C?.1, J?.2 (Pin_2), J?.5 (Pin_5), J?.8 (Pin_8), R?.2, R?.2, R?.2, R?.2, SW?.1, SW?.1, U?.1 (VBAT), U?.1 (Vdd), U?.22 (VSYS), U?.24 (VDD), U?.3 (VOUT), U?.36 (VDDIO2), U?.48 (VDD), U?.5 (V+), U?.5 (VBUS), U?.9 (VDDA)
- new net C245_JUNC: C?.2, J?.2 (Pin_2), R?.1
- new net CC1: J?.A5 (CC1), U?.1 (CC1DB), U?.2 (CC1), U?.4 (I/O3)
- new net CC2: J?.B5 (CC2), U?.4 (CC2), U?.5 (CC2DB), U?.6 (I/O4)
- new net GND: C?.1, C?.2, C?.2, C?.2, C?.2, C?.2, C?.2, C?.2, C?.2, C?.2, C?.2, C?.2, C?.2, C?.2, C?.2, C?.2, C?.2, C?.2, C?.2, D?.2 (A), J?.1 (Pin_1), J?.1 (Pin_1), J?.1 (Pin_1), J?.2 (Pin_2), J?.7 (Pin_7), J?.A1 (GND), J?.A12 (GND), J?.B1 (GND), J?.B12 (GND), J?.S1 (SHIELD), NT?.2, Q?.2 (E), Q?.3 (C), R?.1, R?.1, R?.2, R?.2, R?.2, U?.10 (GND), U?.12 (ADDR0), U?.13 (ADDR1), U?.2 (GND), U?.2 (GND), U?.2 (GND), U?.2 (V-), U?.23 (VSS), U?.25 (GND), U?.3 (GND), U?.3 (SHDN), U?.35 (VSS), U?.47 (VSS), U?.8 (VSSA)
- new net IIN: C?.1, R?.1, U?.10 (PA0), U?.4
- new net INT_N: R?.1, U?.19 (ALERT), U?.25 (PB12)
- new net OLED_SCL: J?.10 (Pin_10), J?.3 (Pin_3), R?.1, U?.42 (PB6), U?.7 (SCL)
- new net OLED_SDA: J?.11 (Pin_11), J?.4 (Pin_4), R?.1, U?.43 (PB7), U?.8 (SDA)
- new net PWM: R?.1, U?.29 (PA8)
- new net SW1: SW?.2, U?.13 (PA3)
- new net SW2: R?.2, SW?.2, U?.2 (PC13), U?.44 (BOOT0)
- new net SWCLK: J?.1 (Pin_1), U?.37 (PA14)
- new net SWDIO: J?.3 (Pin_3), U?.34 (PA13)
- new net TREF: R?.1, U?.15 (PA5)
- new net TTIP: R?.2, U?.11 (PA1)
- new net UIN: C?.1, R?.1, R?.2, U?.12 (PA2)
- new net USB_N: J?.A7 (D-), J?.B7 (D-), U?.1 (I/O1), U?.32 (PA11)
- new net USB_P: J?.A6 (D+), J?.B6 (D+), U?.3 (I/O2), U?.33 (PA12)
- new net VBUS: C?.1, C?.1, F?.1, J?.A4 (VBUS), J?.A9 (VBUS), J?.B4 (VBUS), J?.B9 (VBUS), R?.1, R?.1, R?.1, R?.1, U?.1 (VIN), U?.24 (VDD)
- new net nRST: U?.7 (NRST)
- no-connect marks 0 -> 12
Other:
- note added: "20 (?)"
- note added: "?"

Commit message: Finish schematic, start layouting...
Parts:
- removed Q?: DMP3017SFG, otter:Diodes_PowerDI3333-8, symbol OtterIron_Devkit-rescue:DMP3017SFG-pd-buddy-pd-buddy-sink-rescue-pd-buddy-sink-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
- added J8: +24V, Connector:Banana_Jack_1Pin, symbol Connector:Screw_Terminal_01x01
- added J9: GND, Connector:Banana_Jack_1Pin, symbol Connector:Screw_Terminal_01x01
- added Q4: NCE40P70K or DMP4015SK3Q-13 or IPD50P04P4L11ATMA1, Package_TO_SOT_SMD:TO-252-2, symbol Device:Q_PMOS_GDS
- C1, C10, C12, C13, C14, C15, C2, C4, C6, C7, C8: renamed from C?; footprint otter:C_0603 -> Capacitor_SMD:C_0603_1608Metric
- C11, C16, C17, C18, C19, C22, C3, C5, C9: renamed from C?; footprint otter:C_0402 -> Capacitor_SMD:C_0603_1608Metric
- C20: renamed from C?; footprint otter:CP_Radial_D10.0mm_P5.00mm_flat -> Capacitor_SMD:CP_Elec_10x10.5
- C21: renamed from C?; footprint (none) -> Capacitor_SMD:C_0603_1608Metric
- C23: renamed from C?; footprint (none) -> Capacitor_SMD:CP_Elec_10x10.5
- F1: renamed from F?; value Fuse -> C58066; footprint (none) -> Fuse:Fuseholder_Cylinder-5x20mm_Stelvio-Kontek_PTF78_Horizontal_Open
- J1: renamed from J?; value USB_C_Receptacle_USB2.0 -> C167321; footprint otter:USB-C 16Pin -> Connector_USB:USB_C_Receptacle_Palconn_UTC16-G
- J2: renamed from J?; footprint (none) -> 4mm-banana-test-jack:Test_Jack_4mm
- J3: renamed from J?; value +24V -> GND; footprint (none) -> 4mm-banana-test-jack:Test_Jack_4mm
- J4: renamed from J?; symbol Connector:Conn_01x04_Male -> Connector_Generic:Conn_01x04
- J5: renamed from J?; footprint otter:0.69OLED -> OLED_SSD1306_14pin:OLED_SSD1306_14pin
- J6: renamed from J?; footprint (none) -> Connector_Molex:Molex_KK-254_AE-6410-03A_1x03_P2.54mm_Vertical; symbol Connector:Conn_01x03_Female -> Connector_Generic:Conn_01x03
- J7: renamed from J?; footprint otter:RPC1-12RB-6P(71) -> C245:RPC1-12RB-6P(71)
- R1, R16, R2, R3, R4, R5, R6: renamed from R?; footprint otter:R_0603 -> Resistor_SMD:R_0603_1608Metric
- R10, R11, R12, R13, R14, R15, R17, R18, R20, R21, R22, R23, R7, R8, R9: renamed from R?; footprint otter:R_0402 -> Resistor_SMD:R_0603_1608Metric
- R19: renamed from R?; footprint otter:R_0805 -> Resistor_SMD:R_1206_3216Metric
- U3: renamed from U?; footprint otter:QFN-24-1EP_4x4mm_P0.5mm_EP2.7x2.7mm -> Package_DFN_QFN:QFN-24-1EP_4x4mm_P0.5mm_EP2.7x2.7mm
- U4: renamed from U?; footprint otter:LQFP-48_7x7mm_P0.5mm -> Package_QFP:LQFP-48_7x7mm_P0.5mm
- gave numbers to parts that had none: 13
Connections:
- net GND: now also J9.1 (Pin_1)
- net at C20.1, Q2.3 (C), R11.1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: now also Q4.3 (S)
- net at R16.2: now also Q4.1 (G)
- net at D1.1 (K), L1.1: now also Q4.2 (D)
- net at F1.2, J2.1 (Pin_1): now also J8.1 (Pin_1)
Other:
- note added: "Display: ???"
- note added: "Fuse 5A"
- note added: "Main P-FET:\nDMP3017SFG is discontinued"
- note added: "Option: Cheap chinese\nSSD1306 display module"
- note added: "USB2.0 Type C Receptacle\ne.g. LCSC C167321"
- moved on the sheet: C10, F1, R16

Commit message: Layout draft
Parts:
- added C24: 0.1μF, Capacitor_SMD:C_0603_1608Metric, symbol Device:C
- C20: footprint Capacitor_SMD:CP_Elec_10x10.5 -> Capacitor_THT:CP_Radial_D12.5mm_P5.00mm
- C23: footprint Capacitor_SMD:CP_Elec_10x10.5 -> Capacitor_THT:CP_Radial_D8.0mm_P3.50mm
- R13, R14: symbol Device:R_Small -> Device:R
- SW1, SW2: footprint Button_Switch_SMD:SW_SPST_EVQP7C -> Button_Switch_THT:SW_PUSH_6mm_H13mm
Connections:
- net +3V3: now also C24.1
- net GND: now also C24.2
- net VBUS: now also F1.2, J2.1 (Pin_1), J8.1 (Pin_1); no longer C1.1, F1.1, R13.1, R17.1, R19.1, U1.1 (VIN)
- new net VCC: C1.1, F1.1, R13.1, R17.1, R19.1, U1.1 (VIN)
Other:
- note added: "C20: e.g. 50YXA1000MEFC12.5X25"
- moved on the sheet: C17, R13, R14
Changed lines of the file:
@@
 F 0 "SW2" V 10404 10348 50  0000 L CNN
 F 1 "key1" V 10495 10348 50  0000 L CNN
-F 2 "Button_Switch_SMD:SW_SPST_EVQP7C" H 10450 10400 50  0001 C CNN
+F 2 "Button_Switch_THT:SW_PUSH_6mm_H13mm" H 10450 10400 50  0001 C CNN
 F 3 "" H 10450 10400 50  0001 C CNN
 	1    10450 10200
@@
 F 0 "SW1" V 9604 10348 50  0000 L CNN
 F 1 "key2" V 9695 10348 50  0000 L CNN
-F 2 "Button_Switch_SMD:SW_SPST_EVQP7C" H 9650 10400 50  0001 C CNN
+F 2 "Button_Switch_THT:SW_PUSH_6mm_H13mm" H 9650 10400 50  0001 C CNN
 F 3 "" H 9650 10400 50  0001 C CNN
 	1    9650 10200
@@
 $EndComp
 $Comp
-L power:VBUS #PWR?
-U 1 1 5F199788
-P 1200 9950
-AR Path="/588F9A21/5F199788" Ref="#PWR?"  Part="1"
-AR Path="/588FD270/5F199788" Ref="#PWR?"  Part="1"
-AR Path="/5F199788" Ref="#PWR0127"  Part="1"
-AR Path="/5EFFDF88/5F199788" Ref="#PWR?"  Part="1"
-F 0 "#PWR0127" H 1200 9800 50  0001 C CNN
-F 1 "VBUS" H 1215 10123 50  0000 C CNN
-F 2 "" H 1200 9950 50  0001 C CNN
-F 3 "" H 1200 9950 50  0001 C CNN
-	1    1200 9950
-	1    0    0    -1
-$EndComp
-$Comp
 L power:GND #PWR?
 U 1 1 5F19978E
@@
 $EndComp
 $Comp
-L Device:R_Small R?
+L Device:R R?
 U 1 1 5F1997EA
-P 12200 8950
+P 12200 9100
 AR Path="/5EFFDF88/5F1997EA" Ref="R?"  Part="1"
 AR Path="/5F1997EA" Ref="R14"  Part="1"
-F 0 "R14" H 12259 8996 50  0000 L CNN
-F 1 "100k" H 12259 8905 50  0000 L CNN
-F 2 "Resistor_SMD:R_0603_1608Metric" H 12200 8950 50  0001 C CNN
-F 3 "~" H 12200 8950 50  0001 C CNN
-	1    12200 8950
+F 0 "R14" H 12259 9146 50  0000 L CNN
+F 1 "100k" H 12259 9055 50  0000 L CNN
+F 2 "Resistor_SMD:R_0603_1608Metric" H 12200 9100 50  0001 C CNN
+F 3 "~" H 12200 9100 50  0001 C CNN
+	1    12200 9100
 	-1   0    0    -1
 $EndComp
@@
 L power:GND #PWR?
 U 1 1 5F1997F0
-P 12200 9150
+P 12200 9350
 AR Path="/588FB1D7/5F1997F0" Ref="#PWR?"  Part="1"
 AR Path="/588FD270/5F1997F0" Ref="#PWR?"  Part="1"
 AR Path="/5F1997F0" Ref="#PWR0133"  Part="1"
 AR Path="/5EFFDF88/5F1997F0" Ref="#PWR?"  Part="1"
-F 0 "#PWR0133" H 12200 8900 50  0001 C CNN
-F 1 "GND" H 12205 8977 50  0000 C CNN
-F 2 "" H 12200 9150 50  0001 C CNN
-F 3 "" H 12200 9150 50  0001 C CNN
-	1    12200 9150
+F 0 "#PWR0133" H 12200 9100 50  0001 C CNN
+F 1 "GND" H 12205 9177 50  0000 C CNN
+F 2 "" H 12200 9350 50  0001 C CNN
+F 3 "" H 12200 9350 50  0001 C CNN
+	1    12200 9350
 	-1   0    0    -1
 $EndComp
 Wire Wire Line
-	12200 9050 12200 9150
+	12200 9250 12200 9350
 $Comp
 L Device:C C?
 U 1 1 5F1997F7
-P 12600 9000
+P 12600 9100
 AR Path="/588FB1D7/5F1997F7" Ref="C?"  Part="1"
 AR Path="/588FD270/5F1997F7" Ref="C?"  Part="1"
 AR Path="/5F1997F7" Ref="C17"  Part="1"
 AR Path="/5EFFDF88/5F1997F7" Ref="C?"  Part="1"
-F 0 "C17" H 12715 9046 50  0000 L CNN
-F 1 "0.1μF" H 12715 8955 50  0000 L CNN
-F 2 "Capacitor_SMD:C_0603_1608Metric" H 12638 8850 50  0001 C CNN
-F 3 "~" H 12600 9000 50  0001 C CNN
-	1    12600 9000
+F 0 "C17" H 12715 9146 50  0000 L CNN
+F 1 "0.1μF" H 12715 9055 50  0000 L CNN
+F 2 "Capacitor_SMD:C_0603_1608Metric" H 12638 8950 50  0001 C CNN
+F 3 "~" H 12600 9100 50  0001 C CNN
+	1    12600 9100
 	-1   0    0    -1
 $EndComp
@@
 L power:GND #PWR?
 U 1 1 5F1997FD
-P 12600 9150
+P 12600 9350
 AR Path="/588FB1D7/5F1997FD" Ref="#PWR?"  Part="1"
 AR Path="/588FD270/5F1997FD" Ref="#PWR?"  Part="1"
 AR Path="/5F1997FD" Ref="#PWR0134"  Part="1"
 AR Path="/5EFFDF88/5F1997FD" Ref="#PWR?"  Part="1"
-F 0 "#PWR0134" H 12600 8900 50  0001 C CNN
-F 1 "GND" H 12605 8977 50  0000 C CNN
-F 2 "" H 12600 9150 50  0001 C CNN
-F 3 "" H 12600 9150 50  0001 C CNN
-	1    12600 9150
+F 0 "#PWR0134" H 12600 9100 50  0001 C CNN
+F 1 "GND" H 12605 9177 50  0000 C CNN
+F 2 "" H 12600 9350 50  0001 C CNN
+F 3 "" H 12600 9350 50  0001 C CNN
+	1    12600 9350
 	-1   0    0    -1
 $EndComp
@@
 Connection ~ 12600 8850
 $Comp
-L Device:R_Small R?
+L Device:R R?
 U 1 1 5F199807
-P 12200 8700
+P 12200 8600
 AR Path="/5EFFDF88/5F199807" Ref="R?"  Part="1"
 AR Path="/5F199807" Ref="R13"  Part="1"
-F 0 "R13" H 12259 8746 50  0000 L CNN
-F 1 "560k" H 12259 8655 50  0000 L CNN
-F 2 "Resistor_SMD:R_0603_1608Metric" H 12200 8700 50  0001 C CNN
-F 3 "~" H 12200 8700 50  0001 C CNN
-	1    12200 8700
-	-1   0    0    -1
-$EndComp
-Wire Wire Line
-	12200 8800 12200 8850
-Connection ~ 12200 8850
-$Comp
-L power:VBUS #PWR?
-U 1 1 5F19980F
-P 12200 8600
-AR Path="/588FA3A4/5F19980F" Ref="#PWR?"  Part="1"
-AR Path="/588FD270/5F19980F" Ref="#PWR?"  Part="1"
-AR Path="/5F19980F" Ref="#PWR0135"  Part="1"
-AR Path="/5EFFDF88/5F19980F" Ref="#PWR?"  Part="1"
-F 0 "#PWR0135" H 12200 8450 50  0001 C CNN
-F 1 "VBUS" H 12215 8773 50  0000 C CNN
-F 2 "" H 12200 8600 50  0001 C CNN
-F 3 "" H 12200 8600 50  0001 C CNN
+F 0 "R13" H 12259 8646 50  0000 L CNN
+F 1 "560k" H 12259 8555 50  0000 L CNN
+F 2 "Resistor_SMD:R_0603_1608Metric" H 12200 8600 50  0001 C CNN
+F 3 "~" H 12200 8600 50  0001 C CNN
 	1    12200 8600
 	-1   0    0    -1
@@
 Wire Wire Line
 	5200 10550 4750 10550
-$Comp
-L power:VBUS #PWR?
-U 1 1 5F199835
-P 13100 1050
-AR Path="/588FA5F7/5F199835" Ref="#PWR?"  Part="1"
-AR Path="/588FD270/5F199835" Ref="#PWR?"  Part="1"
-AR Path="/5F199835" Ref="#PWR0136"  Part="1"
-AR Path="/5EFFDF88/5F199835" Ref="#PWR?"  Part="1"
-F 0 "#PWR0136" H 13100 900 50  0001 C CNN
-F 1 "VBUS" H 13115 1223 50  0000 C CNN
-F 2 "" H 13100 1050 50  0001 C CNN
-F 3 "" H 13100 1050 50  0001 C CNN
-	1    13100 1050
-	1    0    0    -1
-$EndComp
 $Comp
 L Amplifier_Operational:OPA340NA U?
@@
 F 0 "C20" H 14038 2246 50  0000 L CNN
 F 1 "1000µF" H 14038 2155 50  0000 L CNN
-F 2 "Capacitor_SMD:CP_Elec_10x10.5" H 13950 2200 50  0001 C CNN
+F 2 "Capacitor_THT:CP_Radial_D12.5mm_P5.00mm" H 13950 2200 50  0001 C CNN
 F 3 "~" H 13950 2200 50  0001 C CNN
 	1    13950 2200
@@
 L power:VBUS #PWR?
 U 1 1 5F9610FB
-P 2050 5750
+P 1550 5600
 AR Path="/588FA5F7/5F9610FB" Ref="#PWR?"  Part="1"
 AR Path="/588FD270/5F9610FB" Ref="#PWR?"  Part="1"
 AR Path="/5F9610FB" Ref="#PWR0148"  Part="1"
 AR Path="/5EFFDFB7/5F9610FB" Ref="#PWR?"  Part="1"
-F 0 "#PWR0148" H 2050 5600 50  0001 C CNN
-F 1 "VBUS" H 2065 5923 50  0000 C CNN
-F 2 "" H 2050 5750 50  0001 C CNN
-F 3 "" H 2050 5750 50  0001 C CNN
-	1    2050 5750
+F 0 "#PWR0148" H 1550 5450 50  0001 C CNN
+F 1 "VBUS" H 1565 5773 50  0000 C CNN
+F 2 "" H 1550 5600 50  0001 C CNN
+F 3 "" H 1550 5600 50  0001 C CNN
+	1    1550 5600
 	1    0    0    -1
 $EndComp
@@
 	1950 5850 2050 5850
 Wire Wire Line
-	2050 5850 2050 5750
+	1550 5700 1550 5600
 Wire Wire Line
 	1450 5850 1550 5850
@@
 F 0 "C23" H 14468 3446 50  0000 L CNN
 F 1 "DNP" H 14468 3355 50  0000 L CNN
-F 2 "Capacitor_SMD:CP_Elec_10x10.5" H 14388 3250 50  0001 C CNN
+F 2 "Capacitor_THT:CP_Radial_D8.0mm_P3.50mm" H 14388 3250 50  0001 C CNN
 F 3 "~" H 14350 3400 50  0001 C CNN
 	1    14350 3400
@@
 Wire Wire Line
 	3800 1250 4900 1250
-Text Notes 14700 2350 0    50   ~ 0
+Text Notes 13450 2850 0    50   ~ 0
 Main P-FET:\nDMP3017SFG is discontinued
 $Comp
@@
 Wire Wire Line
 	1550 6150 2050 6150
+Text Notes 14050 2050 0    50   ~ 0
+C20: e.g. 50YXA1000MEFC12.5X25
+Wire Wire Line
+	12550 6150 12550 6250
+$Comp
+L power:+3V3 #PWR?
+U 1 1 5F07B3FA
+P 12550 5750
+AR Path="/5EFFDF88/5F07B3FA" Ref="#PWR?"  Part="1"
+AR Path="/5F07B3FA" Ref="#PWR0153"  Part="1"
+F 0 "#PWR0153" H 12550 5600 50  0001 C CNN
+F 1 "+3V3" H 12565 5923 50  0000 C CNN
+F 2 "" H 12550 5750 50  0001 C CNN
+F 3 "" H 12550 5750 50  0001 C CNN
+	1    12550 5750
+	1    0    0    -1
+$EndComp
+$Comp
+L power:GND #PWR?
+U 1 1 5F07B400
+P 12550 6250
+AR Path="/5EFFDF88/5F07B400" Ref="#PWR?"  Part="1"
+AR Path="/5F07B400" Ref="#PWR0154"  Part="1"
+F 0 "#PWR0154" H 12550 6000 50  0001 C CNN
+F 1 "GND" H 12555 6077 50  0000 C CNN
+F 2 "" H 12550 6250 50  0001 C CNN
+F 3 "" H 12550 6250 50  0001 C CNN
+	1    12550 6250
+	1    0    0    -1
+$EndComp
+$Comp
+L Device:C C?
+U 1 1 5F07B406
+P 12550 6000
+AR Path="/5EFFDF88/5F07B406" Ref="C?"  Part="1"
+AR Path="/5F07B406" Ref="C24"  Part="1"
+F 0 "C24" H 12665 6046 50  0000 L CNN
+F 1 "0.1μF" H 12665 5955 50  0000 L CNN
+F 2 "Capacitor_SMD:C_0603_1608Metric" H 12588 5850 50  0001 C CNN
+F 3 "~" H 12550 6000 50  0001 C CNN
+	1    12550 6000
+	1    0    0    -1
+$EndComp
+Wire Wire Line
+	12550 5750 12550 5850
+Connection ~ 1550 5700
+$Comp
+L power:VCC #PWR?
+U 1 1 5F1DFA24
+P 2050 5750
+F 0 "#PWR?" H 2050 5600 50  0001 C CNN
+F 1 "VCC" H 2065 5923 50  0000 C CNN
+F 2 "" H 2050 5750 50  0001 C CNN
+F 3 "" H 2050 5750 50  0001 C CNN
+	1    2050 5750
+	1    0    0    -1
+$EndComp
+Wire Wire Line
+	2050 5750 2050 5850
+$Comp
+L power:VCC #PWR?
+U 1 1 5F1F1CDD
+P 1200 9950
+F 0 "#PWR?" H 1200 9800 50  0001 C CNN
+F 1 "VCC" H 1215 10123 50  0000 C CNN
+F 2 "" H 1200 9950 50  0001 C CNN
+F 3 "" H 1200 9950 50  0001 C CNN
+	1    1200 9950
+	1    0    0    -1
+$EndComp
+$Comp
+L power:VCC #PWR?
+U 1 1 5F1F2D8D
+P 12200 8350
+F 0 "#PWR?" H 12200 8200 50  0001 C CNN
+F 1 "VCC" H 12215 8523 50  0000 C CNN
+F 2 "" H 12200 8350 50  0001 C CNN
+F 3 "" H 12200 8350 50  0001 C CNN
+	1    12200 8350
+	1    0    0    -1
+$EndComp
+Wire Wire Line
+	12200 8950 12200 8850
+Connection ~ 12200 8850
+Wire Wire Line
+	12200 8750 12200 8850
+Wire Wire Line
+	12200 8450 12200 8350
+Wire Wire Line
+	12600 8950 12600 8850
+Wire Wire Line
+	12600 9250 12600 9350
+$Comp
+L power:VCC #PWR?
+U 1 1 5F27296C
+P 13100 1050
+F 0 "#PWR?" H 13100 900 50  0001 C CNN
+F 1 "VCC" H 13115 1223 50  0000 C CNN
+F 2 "" H 13100 1050 50  0001 C CNN
+F 3 "" H 13100 1050 50  0001 C CNN
+	1    13100 1050
+	1    0    0    -1
+$EndComp
 $EndSCHEMATC
